File: Arduino_Nano_UV_Box_4-Digit_7-Seg_CC_sch/Arduino_Nano_Countdown_Timer_7-seg_CC.brd (EAGLE design)
At the start: 104.1 x 45.7 mm, 34 parts, among them M2 ARDUINO-NANO-3.0, Q1 IRL540, T1 PN2222A, T2 PN2222A, T3 PN2222A, T4 PN2222A

Commit message: Add files via upload
Parts:
- LED: value Plue -> Blue
Changed lines of the file:
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@@
 <attribute name="VALUE" x="11.698840625" y="35.39405625" size="0.6096" layer="28" ratio="10" rot="MR0"/>
 </element>
-<element name="LED" library="1_My_Library" package="LED3MM" value="Plue" x="11.43" y="33.02" smashed="yes" rot="R180">
+<element name="LED" library="1_My_Library" package="LED3MM" value="Blue" x="11.43" y="33.02" smashed="yes" rot="R180">
 <attribute name="NAME" x="10.16" y="28.956" size="1.016" layer="25" ratio="10"/>
 <attribute name="VALUE" x="10.16" y="26.9875" size="1.016" layer="27" ratio="10"/>
