File: Arduino_Nano_UV_Box_4-Digit_7-Seg_CC_sch/Arduino_Nano_Countdown_Timer_7-seg_CC.sch (EAGLE design)
At the start: 34 parts, among them M2 ARDUINO-NANO-3.0, Q1 IRL540, T1 PN2222A, T2 PN2222A, T3 PN2222A, T4 PN2222A

Commit message: Add files via upload
Parts:
- LED: value Plue -> Blue
Changed lines of the file:
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@@
 <part name="Q1" library="transistor-power" library_urn="urn:adsk.eagle:library:400" deviceset="IRF540" device="" package3d_urn="urn:adsk.eagle:package:29484/3" value="IRL540"/>
 <part name="R15" library="1_My_Library" deviceset="RESISTOR" device="R0805" value="2k2"/>
-<part name="LED" library="1_My_Library" deviceset="LED" device="3MM" value="Plue"/>
+<part name="LED" library="1_My_Library" deviceset="LED" device="3MM" value="Blue"/>
 <part name="SUPPLY10" library="1_Stavros" deviceset="+12V" device=""/>
 <part name="SUPPLY23" library="1_Stavros" deviceset="0V" device=""/>
