File: Schematics/Arduino_Nano_Countdown_Timer_7-seg_CC.brd (EAGLE design)
At the start: 104.1 x 45.7 mm, 34 parts, among them M2 ARDUINO-NANO-3.0, Q1 IRL540, T1 PN2222A, T2 PN2222A, T3 PN2222A, T4 PN2222A

Commit message: Add files via upload
Parts:
- C5: device 1_Stavros:E5-6.5 -> 1_My_Library:E5-6.5
- C6: device 1_Stavros:C050-025X075 -> 1_My_Library:C050-025X075
- D2: device 1_Stavros:DO41-10 -> 1_My_Library:DO41-10
- DOWN, START, UP: device 1_Stavros:DTE6K -> 1_My_Library:DTE6K
- LOAD, PWR: device Connector-Molex_Stavros:22-23-2021 -> My_Connector-Molex:22-23-2021
- PAUSE: device MY_Switch-misc:2PIN_HEADER -> My_Switch-misc:2PIN_HEADER
- R17: device 1_Stavros:R0805 -> 1_My_Library:R0805
- moved R17 0.32 mm to (18.7, 30.5)
Connections:
- net 0V renamed GND
Routing:
- net GND: track 328.4 -> 325.8 mm
