File: Schematics/Arduino_Nano_Countdown_Timer_7-seg_CC.sch (EAGLE design)
At the start: 34 parts, among them M2 ARDUINO-NANO-3.0, Q1 IRL540, T1 PN2222A, T2 PN2222A, T3 PN2222A, T4 PN2222A

Commit message: Add files via upload
Parts:
- C5: device 1_Stavros:CAPACITOR_POLE5-6.5 -> 1_My_Library:CAPACITOR_POLE5-6.5
- C6: device 1_Stavros:CAPACITOR050-025X075 -> 1_My_Library:CAPACITOR050-025X075
- D2: device 1_Stavros:DIODE1N4004 -> 1_My_Library:DIODE1N4004
- DOWN, START, UP: device 1_Stavros:SWITCHE6K -> 1_My_Library:SWITCHE6K
- LOAD, PWR: device Connector-Molex_Stavros:22-23-2021 -> My_Connector-Molex:22-23-2021
- PAUSE: device MY_Switch-misc:REED-SWITCH-2PIN -> My_Switch-misc:REED-SWITCH-2PIN
- R17: device 1_Stavros:RESISTORR0805 -> 1_My_Library:RESISTORR0805
Connections:
- net 0V renamed GND
